Commit message: update

File: install/arm_description/share/arm_description/urdf/arm.urdf (robot description, URDF)
Before this commit: robot agbot_arm, 20 links, 19 joints
Links:
- removed link arm_rgb_camera
- removed link arm_rgb_camera_optical
- removed link base_plate
- removed link claw_support
- removed link elbow
- removed link forward_drive_arm
- removed link gripper_left
- removed link gripper_right
- removed link horizontal_arm
- removed link wrist
- added link arm_rgb_camera_link, mass 0.001; collision mesh filename=file:///home/albert/rad_ws/install/agbot_full_description/s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 scale=0.002 0.002 0.002; visual mesh filename=file:///home/albert/rad_ws/install/agbot_full_description/s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 scale=0.002 0.002 0.002
- added link arm_rgb_camera_optical_link
- added link base_plate_link, mass 0.1; collision mesh filename=file:///home/albert/rad_ws/install/agbot_description/share/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 scale=0.0015 0.0015 0.002; visual mesh filename=file:///home/albert/rad_ws/install/agbot_description/share/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 scale=0.0015 0.0015 0.002
- added link claw_support_link, mass 0.05; collision mesh filename=file:///home/albert/rad_ws/install/agbot_full_description/s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 scale=0.004 0.004 0.004; visual mesh filename=file:///home/albert/rad_ws/install/agbot_full_description/s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 scale=0.004 0.004 0.004
- added link elbow_link, mass 0.05; collision cylinder length=0.18 radius=0.015; visual cylinder length=0.18 radius=0.015
- added link forward_drive_arm_link, mass 0.1; collision box size=0.75 0.05 0.005; visual box size=0.75 0.05 0.005
- added link gripper_left_link, mass 0.01; collision mesh filename=file:///home/albert/rad_ws/install/agbot_full_description/s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 scale=0.004 0.004 0.004; visual mesh filename=file:///home/albert/rad_ws/install/agbot_full_description/s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 scale=0.004 0.004 0.004
- added link gripper_right_link, mass 0.01; collision mesh filename=file:///home/albert/rad_ws/install/agbot_full_description/s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 scale=0.004 0.004 0.004; visual mesh filename=file:///home/albert/rad_ws/install/agbot_full_description/s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 scale=0.004 0.004 0.004
- added link horizontal_arm_link, mass 0.1; collision box size=0.555 0.05 0.005; visual box size=0.555 0.05 0.005
- added link wrist_link, mass 0.05; collision cylinder length=0.18 radius=0.015; visual cylinder length=0.09 radius=0.015
Joints:
- joint body_arm_joint: parent roboball_cylinder -> roboball_cylinder_link
- joint robo_cylinder_joint: child roboball_cylinder -> roboball_cylinder_link

File: install/arm_description/share/arm_description/urdf/arm.xacro (robot description, xacro)
@@ -74,5 +74,5 @@
     <link name = "world">
     </link>
-    <link name = "roboball_cylinder">
+    <link name = "roboball_cylinder_link">
         <visual>
             <geometry>
@@ -181,5 +181,5 @@
         </collision>
     </link>
-    <link name="base_plate">
+    <link name="base_plate_link">
         <xacro:default_inertia mass="0.1"/>
          <visual>
@@ -197,5 +197,5 @@
         </collision>
     </link>
-    <link name="forward_drive_arm">
+    <link name="forward_drive_arm_link">
         <xacro:default_inertia mass="0.1"/>
         <visual>
@@ -213,5 +213,5 @@
         </collision>
     </link>
-    <link name = "elbow">
+    <link name = "elbow_link">
         <visual>
             <origin xyz="0 0 0" rpy="0 ${PI / 2} 0"/>
@@ -230,5 +230,5 @@
                                 xyz = "0 0 0" rpy = "0 0 0"/>
     </link>
-    <link name="horizontal_arm">
+    <link name="horizontal_arm_link">
         <xacro:default_inertia mass="0.1"/>
         <visual>
@@ -246,5 +246,5 @@
         </collision>
     </link>
-    <link name = "wrist">
+    <link name = "wrist_link">
         <visual>
             <origin xyz="0 0 0" rpy="0 ${PI / 2} 0"/>
@@ -263,5 +263,5 @@
                                 xyz = "0 0 0" rpy = "0 0 0"/>
     </link>
-    <link name="claw_support">
+    <link name="claw_support_link">
         <xacro:default_inertia mass="0.05"/>
         <visual>
@@ -279,5 +279,5 @@
         </collision>
     </link>
-    <link name="gripper_right">
+    <link name="gripper_right_link">
         <xacro:default_inertia mass="0.01"/>
         <visual>
@@ -295,5 +295,5 @@
         </collision>
     </link>
-    <link name="gripper_left">
+    <link name="gripper_left_link">
         <xacro:default_inertia mass="0.01"/>
         <visual>
@@ -311,7 +311,7 @@
         </collision>
     </link>
-    <link name="arm_rgb_camera_optical" >
-    </link>
-    <link name="arm_rgb_camera">
+    <link name="arm_rgb_camera_optical_link" >
+    </link>
+    <link name="arm_rgb_camera_link">
         <xacro:default_inertia mass="0.001"/>
         <visual>
@@ -332,11 +332,12 @@
     <joint name = "robo_cylinder_joint" type = "fixed">
         <parent link="world" />
-        <child link="roboball_cylinder" />
+        <child link="roboball_cylinder_link" />
         <origin xyz = "0 0 ${base_height + robo_cylinder_radius}" rpy = "${PI/2} 0 0" />
      </joint>
      <joint name = "body_arm_joint" type = "fixed">
-        <parent link="world" />
+        <parent link="roboball_cylinder_link" />
         <child link="arm_base_rail_link" />
-        <origin xyz = "0 0 ${3*arm_base_rail_height}" rpy = "0 0 ${PI/2}" />
+        <!-- <origin xyz = "0 0 ${3*arm_base_rail_height}" rpy = "0 ${PI/2} ${PI/2}" />       -->
+        <origin xyz = "0 -${robo_cylinder_radius - (5*arm_base_rail_height)} 0" rpy = "0 ${PI/2} ${PI/2}" />
      </joint>
      <joint name = "base_rail_to_ mid_rail_joint" type = "prismatic">
@@ -380,5 +381,5 @@
     <joint name ="arm_base_joint" type="revolute">
         <parent link="arm_base_link"/>
-        <child link = "base_plate"/>
+        <child link = "base_plate_link"/>
         <origin xyz="0 0 0.07"/>
         <axis xyz="0 0 1"/>
@@ -387,6 +388,6 @@
     </joint>
     <joint name="shoulder_joint" type="revolute">
-        <parent link="base_plate"/>
-        <child link="forward_drive_arm"/>
+        <parent link="base_plate_link"/>
+        <child link="forward_drive_arm_link"/>
         <origin xyz="0 0 0.075" rpy="-${PI/2} 0 0"/>
         <axis xyz="1 0 0"/>
@@ -394,11 +395,11 @@
     </joint>
     <joint name = "shoulder_elbow_joint" type = "fixed">
-        <parent link = "forward_drive_arm"/>
-        <child link = "elbow"/>
+        <parent link = "forward_drive_arm_link"/>
+        <child link = "elbow_link"/>
         <origin xyz = "${(forward_drive_arm_width / 1.5) + 0.02} 0 ${forward_drive_arm_length}" rpy = "0 0 0"/>
     </joint>
     <joint name="elbow_joint" type="revolute">
-        <parent link="elbow"/>
-        <child link="horizontal_arm"/>
+        <parent link="elbow_link"/>
+        <child link="horizontal_arm_link"/>
         <origin xyz="${cylinder_length/4} 0 0" rpy="-${PI} 0 0"/>
         <axis xyz="1 0 0"/>
@@ -406,11 +407,11 @@
     </joint>
     <joint name = "elbow_forearm_joint" type = "fixed">
-        <parent link = "horizontal_arm"/>
-        <child link = "wrist"/>
+        <parent link = "horizontal_arm_link"/>
+        <child link = "wrist_link"/>
         <origin xyz = "0 0 ${horizontal_arm_length}" rpy = "0 0 0"/>
     </joint>
     <joint name="wrist_joint" type="revolute">
-        <parent link="wrist"/>
-        <child link="claw_support"/>
+        <parent link="wrist_link"/>
+        <child link="claw_support_link"/>
         <origin xyz="0 0 0" />
         <axis xyz="1 0 0"/>
@@ -418,6 +419,6 @@
     </joint>
     <joint name="gripper_right_joint" type="revolute">
-        <parent link="claw_support"/>
-        <child link="gripper_right"/>
+        <parent link="claw_support_link"/>
+        <child link="gripper_right_link"/>
         <origin xyz="-0.037 -0.015 0.083"/>
         <axis xyz="0 1 0"/>
@@ -426,6 +427,6 @@
     <joint name="gripper_left_joint" type="revolute">
         <mimic joint="gripper_right_joint" multiplier="-1"/>
-        <parent link="claw_support"/>
-        <child link="gripper_left"/>
+        <parent link="claw_support_link"/>
+        <child link="gripper_left_link"/>
         <origin xyz="0.042 -0.015 0.083"/>
         <axis xyz="0 1 0"/>
@@ -433,11 +434,11 @@
     </joint>
     <joint name="arm_camera_optical_joint" type="fixed">
-        <parent link="claw_support"/>
-        <child link="arm_rgb_camera_optical"/>
+        <parent link="claw_support_link"/>
+        <child link="arm_rgb_camera_optical_link"/>
         <origin xyz = "0 .10 0.085" rpy = "0 0 0" />
     </joint>
     <joint name = "arm_rgb_camera_joint" type = "fixed" >
-        <parent link = "arm_rgb_camera_optical" />
-        <child link = "arm_rgb_camera" />
+        <parent link = "arm_rgb_camera_optical_link" />
+        <child link = "arm_rgb_camera_link" />
         <origin xyz="0 0 0.03" rpy="0 -${PI/2} 0"/>
     </joint>

File: install/arm_description/share/arm_description/urdf/arm_gazebo.xacro (robot description, xacro)
@@ -10,5 +10,5 @@
       </plugin>
     </gazebo>
-      <gazebo reference="arm_rgb_camera">
+      <gazebo reference="arm_rgb_camera_link">
         <sensor name="camera_sensor" type="camera">
           <pose>0 0 0 0 0 0</pose>
@@ -32,5 +32,5 @@
         </sensor>
       </gazebo>
-    <gazebo reference = "roboball_cylinder">
+    <gazebo reference = "roboball_cylinder_link">
       <material>Gazebo/GreyTransparent</material>
       <mu1>30.0</mu1>
@@ -61,26 +61,26 @@
         <material>Gazebo/Blue</material>
       </gazebo>
-      <gazebo reference="base_plate">
+      <gazebo reference="base_plate_link">
         <material>Gazebo/Red</material>
       </gazebo>
-      <gazebo reference="forward_drive_arm">
+      <gazebo reference="forward_drive_arm_link">
         <material>Gazebo/Yellow</material>
       </gazebo>
-      <gazebo reference="elbow">
+      <gazebo reference="elbow_link">
         <material>Gazebo/White</material>
       </gazebo>
-      <gazebo reference="horizontal_arm">
+      <gazebo reference="horizontal_arm_link">
         <material>Gazebo/Green</material>
       </gazebo>
-      <gazebo reference="claw_support">
+      <gazebo reference="claw_support_link">
         <material>Gazebo/Yellow</material>
       </gazebo>
-      <gazebo reference="gripper_right">
+      <gazebo reference="gripper_right_link">
         <material>Gazebo/Purple</material>
       </gazebo>
-      <gazebo reference="gripper_left">
+      <gazebo reference="gripper_left_link">
         <material>Gazebo/Purple</material>
       </gazebo>
-      <gazebo reference="arm_rgb_camera">
+      <gazebo reference="arm_rgb_camera_link">
         <material>Gazebo/Blue</material>
       </gazebo>

File: install/arm_setup_moveit/share/arm_setup_moveit/config/agbot_arm.ros2_control.xacro (robot description, xacro)
@@ -8,18 +8,4 @@
                 <plugin>mock_components/GenericSystem</plugin>
             </hardware>
-            <joint name="wrist_joint">
-                <command_interface name="position"/>
-                <state_interface name="position">
-                  <param name="initial_value">${initial_positions['wrist_joint']}</param>
-                </state_interface>
-                <state_interface name="velocity"/>
-            </joint>
-            <joint name="gripper_right_joint">
-                <command_interface name="position"/>
-                <state_interface name="position">
-                  <param name="initial_value">${initial_positions['gripper_right_joint']}</param>
-                </state_interface>
-                <state_interface name="velocity"/>
-            </joint>
             <joint name="base_rail_to_ mid_rail_joint">
                 <command_interface name="position"/>
@@ -57,4 +43,18 @@
                 <state_interface name="velocity"/>
             </joint>
+            <joint name="wrist_joint">
+                <command_interface name="position"/>
+                <state_interface name="position">
+                  <param name="initial_value">${initial_positions['wrist_joint']}</param>
+                </state_interface>
+                <state_interface name="velocity"/>
+            </joint>
+            <joint name="gripper_right_joint">
+                <command_interface name="position"/>
+                <state_interface name="position">
+                  <param name="initial_value">${initial_positions['gripper_right_joint']}</param>
+                </state_interface>
+                <state_interface name="velocity"/>
+            </joint>
         </ros2_control>
     </xacro:macro>

Commit message: Added Moveit2 API module.

File: install/arm_description/share/arm_description/urdf/arm.urdf (robot description, URDF)
Before this commit: robot agbot_arm, 20 links, 19 joints
Links:
- removed link roboball_cylinder
Joints:
- removed joint robo_cylinder_joint
- joint body_arm_joint: parent roboball_cylinder_link -> world

File: install/arm_description/share/arm_description/urdf/arm.xacro (robot description, xacro)
@@ -13,6 +13,6 @@
     <xacro:property name="scale" value="0.0025 0.0025 0.0025"/>
     <xacro:property name="arm_scale" value="0.0015 0.0015 0.002"/>
-    <xacro:property name="claw_scale" value="0.004 0.004 0.004"/>
-    <xacro:property name="claw_camera_scale" value="0.002 0.002 0.002"/>
+    <xacro:property name="claw_scale" value="0.003 0.003 0.003"/>
+    <xacro:property name="claw_camera_scale" value="0.001 0.001 0.001"/>
     <xacro:property name="base_height" value="0.0" />
     <xacro:property name = "forward_drive_arm_length" value = "0.75" />
@@ -74,5 +74,5 @@
     <link name = "world">
     </link>
-    <link name = "roboball_cylinder_link">
+    <!-- <link name = "roboball_cylinder_link">
         <visual>
             <geometry>
@@ -90,5 +90,5 @@
         <xacro:cylinder_inertia m = "3.0" r = "${robo_cylinder_radius}" h = "${robo_cylinder_length}"
                                 xyz = "0 0 0" rpy = "0 0 0"/>
-    </link>
+    </link> -->
     <link name="arm_base_rail_link">
         <visual>
@@ -330,19 +330,20 @@
     </link>
     <!-- Joint Descriptions -->
-    <joint name = "robo_cylinder_joint" type = "fixed">
+    <!-- <joint name = "robo_cylinder_joint" type = "fixed">
         <parent link="world" />
         <child link="roboball_cylinder_link" />
         <origin xyz = "0 0 ${base_height + robo_cylinder_radius}" rpy = "${PI/2} 0 0" />
-     </joint>
+     </joint>    -->
      <joint name = "body_arm_joint" type = "fixed">
-        <parent link="roboball_cylinder_link" />
+        <!-- <parent link="roboball_cylinder_link" /> -->
+        <parent link="world" />
         <child link="arm_base_rail_link" />
-        <!-- <origin xyz = "0 0 ${3*arm_base_rail_height}" rpy = "0 ${PI/2} ${PI/2}" />       -->
-        <origin xyz = "0 -${robo_cylinder_radius - (5*arm_base_rail_height)} 0" rpy = "0 ${PI/2} ${PI/2}" />
+        <!-- <origin xyz = "0 -${robo_cylinder_radius - (5*arm_base_rail_height)} 0" rpy = "0 ${PI/2} ${PI/2}" /> -->
+        <origin xyz = "0 -${robo_cylinder_radius - (5*arm_base_rail_height)} 0" rpy = "0 0 0" />
      </joint>
      <joint name = "base_rail_to_ mid_rail_joint" type = "prismatic">
         <parent link = "arm_base_rail_link"/>
         <child link="arm_mid_rail_link" />
-        <origin xyz = "0 0 ${arm_base_rail_height}" rpy = "0 0 0" />
+        <origin xyz = "0 0 ${arm_base_rail_height + 0.001}" rpy = "0 0 0" />
         <limit lower="0" upper="${((arm_base_rail_length / 2) + (arm_base_rail_length / 4))/2}" effort="100.0" velocity="0.5"/>
      </joint>
@@ -350,20 +351,20 @@
         <parent link = "arm_base_car_link"/>
         <child link = "box_one_link" />
-        <origin xyz = "-${(arm_base_rail_length / 2) - (box_length / 2)} 0 ${arm_base_rail_height}" rpy = "0 0 0"/>
+        <origin xyz = "-${(arm_base_rail_length / 2) - (box_length / 2)} 0 ${arm_base_rail_height + .001}" rpy = "0 0 0"/>
      </joint>
      <joint name = "box_two_joint" type = "fixed">
         <parent link = "arm_base_car_link"/>
         <child link = "box_two_link" />
-        <origin xyz = "-${(arm_base_rail_length / 2) - (box_length * 1.5) - 0.05} 0 ${arm_base_rail_height}" rpy = "0 0 0"/>
+        <origin xyz = "-${(arm_base_rail_length / 2) - (box_length * 1.5) - 0.05} 0 ${arm_base_rail_height + .001}" rpy = "0 0 0"/>
      </joint>
      <joint name = "box_three_joint" type = "fixed">
         <parent link = "arm_base_car_link"/>
         <child link = "box_three_link" />
-        <origin xyz = "${(box_length / 2) - 0.05} 0 ${arm_base_rail_height}" rpy = "0 0 0"/>
+        <origin xyz = "${(box_length / 2) - 0.05} 0 ${arm_base_rail_height + .001}" rpy = "0 0 0"/>
      </joint>
      <joint name = "box_four_joint" type = "fixed">
         <parent link = "arm_base_car_link"/>
         <child link = "box_four_link" />
-        <origin xyz = "${box_length *1.5} 0 ${arm_base_rail_height}" rpy = "0 0 0"/>
+        <origin xyz = "${box_length *1.5} 0 ${arm_base_rail_height + .001}" rpy = "0 0 0"/>
      </joint>
     <!-- Robot Arm -->
@@ -371,5 +372,5 @@
         <parent link = "arm_mid_rail_link"/>
         <child link = "arm_base_car_link"/>
-        <origin xyz = "0 0 ${arm_base_rail_height}" rpy = "0 0 0"/>
+        <origin xyz = "0 0 ${arm_base_rail_height + 0.001}" rpy = "0 0 0"/>
         <limit lower="0" upper="${(arm_base_rail_length / 2) + (arm_base_rail_length / 4)}" effort="100.0" velocity="0.5"/>
     </joint>
@@ -377,12 +378,12 @@
         <parent link = "arm_base_car_link"/>
         <child link = "arm_base_link"/>
-        <origin xyz = "${(arm_base_rail_length / 2) - (arm_base_rail_length / 20)} 0 ${arm_base_car_height}" rpy = "0 0 ${PI/2}"/>
+        <origin xyz = "${(arm_base_rail_length / 2) - (arm_base_rail_length / 20)} -0.02 ${arm_base_car_height+.002}" rpy = "0 0 ${PI/2}"/>
     </joint>
     <joint name ="arm_base_joint" type="revolute">
         <parent link="arm_base_link"/>
         <child link = "base_plate_link"/>
-        <origin xyz="0 0 0.07"/>
+        <origin xyz="0 0 0.072" />
         <axis xyz="0 0 1"/>
-        <limit lower="-${PI}" upper="${PI}"
+        <limit lower="0" upper="${PI}"
                effort="${effort}" velocity="${velocity}"/>
     </joint>
@@ -397,10 +398,10 @@
         <parent link = "forward_drive_arm_link"/>
         <child link = "elbow_link"/>
-        <origin xyz = "${(forward_drive_arm_width / 1.5) + 0.02} 0 ${forward_drive_arm_length}" rpy = "0 0 0"/>
+        <origin xyz = "${(forward_drive_arm_width / 1.5) + 0.02} 0 ${forward_drive_arm_length + 0.022}" rpy = "0 0 0"/>
     </joint>
     <joint name="elbow_joint" type="revolute">
         <parent link="elbow_link"/>
         <child link="horizontal_arm_link"/>
-        <origin xyz="${cylinder_length/4} 0 0" rpy="-${PI} 0 0"/>
+        <origin xyz="${cylinder_length/4} 0 -0.022" rpy="-${PI} 0 0"/>
         <axis xyz="1 0 0"/>
         <limit lower="-${PI}" upper="0" effort="${effort}" velocity="${velocity}"/>
@@ -409,10 +410,10 @@
         <parent link = "horizontal_arm_link"/>
         <child link = "wrist_link"/>
-        <origin xyz = "0 0 ${horizontal_arm_length}" rpy = "0 0 0"/>
+        <origin xyz = "0 0 ${horizontal_arm_length + 0.02}" rpy = "0 0 0"/>
     </joint>
     <joint name="wrist_joint" type="revolute">
         <parent link="wrist_link"/>
         <child link="claw_support_link"/>
-        <origin xyz="0 0 0" />
+        <origin xyz="0 0 0.02" />
         <axis xyz="1 0 0"/>
         <limit lower="-${PI / 2}" upper="${PI / 2}" effort="${effort}" velocity="${velocity}"/>
@@ -421,5 +422,5 @@
         <parent link="claw_support_link"/>
         <child link="gripper_right_link"/>
-        <origin xyz="-0.037 -0.015 0.083"/>
+        <origin xyz="-0.046 -0.013 0.014"/>
         <axis xyz="0 1 0"/>
         <limit lower="-${PI / 2}" upper="0.0" effort="${effort}" velocity="${velocity}"/>
@@ -429,5 +430,5 @@
         <parent link="claw_support_link"/>
         <child link="gripper_left_link"/>
-        <origin xyz="0.042 -0.015 0.083"/>
+        <origin xyz="0.015 -0.013 0.014"/>
         <axis xyz="0 1 0"/>
         <limit lower="0.0" upper="${PI / 2}" effort="${effort}" velocity="${velocity}"/>

File: install/arm_description/share/arm_description/urdf/arm_gazebo.xacro (robot description, xacro)
@@ -32,9 +32,9 @@
         </sensor>
       </gazebo>
-    <gazebo reference = "roboball_cylinder_link">
+    <!-- <gazebo reference = "roboball_cylinder_link">
       <material>Gazebo/GreyTransparent</material>
       <mu1>30.0</mu1>
       <mu2>30.0</mu2>
-    </gazebo>
+    </gazebo> -->
     <gazebo reference="arm_base_rail_link">
         <material>Gazebo/White</material>

File: install/arm_description/share/arm_description/urdf/arm_ros2_control.xacro (robot description, xacro)
@@ -14,6 +14,4 @@
             </command_interface>
             <state_interface name="position"/>
-            <!-- <state_interface name="velocity"/>
-            <state_interface name="effort"/> -->
         </joint>
         <joint name="mid_rail_to_arm_car_joint">
@@ -23,10 +21,8 @@
             </command_interface>
             <state_interface name="position"/>
-            <!-- <state_interface name="velocity"/>
-            <state_interface name="effort"/> -->
         </joint>
         <joint name="arm_base_joint">
             <command_interface name="position">
-                <param name="min">-${PI}</param>
+                <param name="min">0</param>
                 <param name="max">${PI}</param>
             </command_interface>
@@ -36,5 +32,5 @@
             <command_interface name="position">
                 <param name="min">0</param>
-                <param name="max">4</param>
+                <param name="max">${PI}</param>
             </command_interface>
             <state_interface name="position"/>
@@ -56,10 +52,8 @@
         <joint name="gripper_right_joint">
             <command_interface name="position">
-            <!-- <command_interface name="effort"> -->
                 <param name="min">-${(PI/2)+.01}</param>
                 <param name="max">0.01</param>
             </command_interface>
             <state_interface name="position"/>
-            <!-- <state_interface name="effort"/> -->
         </joint>
         <joint name="gripper_left_joint">
@@ -67,5 +61,4 @@
             <param name="multiplier">-1</param>
             <command_interface name="position">
-            <!-- <command_interface name="effort"> -->
                 <param name="min">-0.01</param>
                 <param name="max">${PI/2}</param>
