Commit message: Added Alexa Voice Interface support.

File: install/arm_description/share/arm_description/urdf/arm.xacro (robot description, xacro)
@@ -383,7 +383,7 @@
         <parent link="arm_base_link"/>
         <child link = "base_plate_link"/>
-        <origin xyz="0 0 0.072" />
+        <origin xyz="0 0 0.072" rpy = "0 0 0"/>
         <axis xyz="0 0 1"/>
-        <limit lower="0" upper="${PI}"
+        <limit lower="-${PI/2}" upper="${PI/2}"
                effort="${effort}" velocity="${velocity}"/>
     </joint>
@@ -393,5 +393,5 @@
         <origin xyz="0 0 0.075" rpy="-${PI/2} 0 0"/>
         <axis xyz="1 0 0"/>
-        <limit lower="0" upper="4.0" effort="${effort}" velocity="${velocity}"/>
+        <limit lower="0" upper="${PI}" effort="${effort}" velocity="${velocity}"/>
     </joint>
     <joint name = "shoulder_elbow_joint" type = "fixed">

File: install/arm_description/share/arm_description/urdf/arm_ros2_control.xacro (robot description, xacro)
@@ -24,6 +24,6 @@
         <joint name="arm_base_joint">
             <command_interface name="position">
-                <param name="min">0</param>
-                <param name="max">${PI}</param>
+                <param name="min">-${PI/2}</param>
+                <param name="max">${PI/2}</param>
             </command_interface>
             <state_interface name="position"/>

Commit message: Added video of Alexa interface

File: install/arm_description/share/arm_description/urdf/arm.xacro (robot description, xacro)
@@ -47,5 +47,4 @@
     <xacro:macro name="default_transmission" params="name">
         <transmission name="transmission_${name}">
-            <!-- <plugin>transmission_interface/DifferentialTransmission</plugin> -->
             <plugin>transmission_interface/SimpleTransmission</plugin>
             <actuator name="motor_${name}" role="actuator1"/>
@@ -74,5 +73,5 @@
     <link name = "world">
     </link>
-    <!-- <link name = "roboball_cylinder_link">
+    <link name = "roboball_cylinder_link">
         <visual>
             <geometry>
@@ -90,5 +89,5 @@
         <xacro:cylinder_inertia m = "3.0" r = "${robo_cylinder_radius}" h = "${robo_cylinder_length}"
                                 xyz = "0 0 0" rpy = "0 0 0"/>
-    </link> -->
+    </link>
     <link name="arm_base_rail_link">
         <visual>
@@ -330,15 +329,15 @@
     </link>
     <!-- Joint Descriptions -->
-    <!-- <joint name = "robo_cylinder_joint" type = "fixed">
+    <joint name = "robo_cylinder_joint" type = "fixed">
         <parent link="world" />
         <child link="roboball_cylinder_link" />
         <origin xyz = "0 0 ${base_height + robo_cylinder_radius}" rpy = "${PI/2} 0 0" />
-     </joint>    -->
+     </joint>
      <joint name = "body_arm_joint" type = "fixed">
-        <!-- <parent link="roboball_cylinder_link" /> -->
-        <parent link="world" />
+        <parent link="roboball_cylinder_link" />
+        <!-- <parent link="world" /> -->
         <child link="arm_base_rail_link" />
-        <!-- <origin xyz = "0 -${robo_cylinder_radius - (5*arm_base_rail_height)} 0" rpy = "0 ${PI/2} ${PI/2}" /> -->
-        <origin xyz = "0 -${robo_cylinder_radius - (5*arm_base_rail_height)} 0" rpy = "0 0 0" />
+        <origin xyz = "0 -${robo_cylinder_radius - (5*arm_base_rail_height)} 0" rpy = "0 ${PI/2} ${PI/2}" />
+        <!-- <origin xyz = "0 -${robo_cylinder_radius - (5*arm_base_rail_height)} 0" rpy = "0 0 0" /> -->
      </joint>
      <joint name = "base_rail_to_ mid_rail_joint" type = "prismatic">

File: install/arm_description/share/arm_description/urdf/arm_gazebo.xacro (robot description, xacro)
@@ -32,9 +32,9 @@
         </sensor>
       </gazebo>
-    <!-- <gazebo reference = "roboball_cylinder_link">
+    <gazebo reference = "roboball_cylinder_link">
       <material>Gazebo/GreyTransparent</material>
       <mu1>30.0</mu1>
       <mu2>30.0</mu2>
-    </gazebo> -->
+    </gazebo>
     <gazebo reference="arm_base_rail_link">
         <material>Gazebo/White</material>
